File: 4201_multiples_kicad/4201_multiples.kicad_pcb (KiCad board)
At the start: 2 copper layers, 60 x 110 mm, 74 parts, among them J1 PJ392, J10 Conn_01x04_Female, J11 Conn_01x05_Female, J12 Conn_01x04_Female, J13 Conn_01x04_Female, J14 Conn_01x05_Male, J15 Conn_01x04_Male, J16 Conn_01x05_Male, J17 Conn_01x04_Male, J18 Conn_01x04_Male, J19 Conn_02x05_Odd_Even, J2 PJ392, J3 PJ392, J4 PJ392, J5 PJ392, J6 PJ392, J7 PJ392, J8 PJ392, J9 Conn_01x05_Female, U1 TL074, U2 TL074

Commit message: Set LED resistor values and change ICs to LM324
Parts:
- D13, D14: value Schottky -> LL103A
- D4: value green -> 1.8mm_green
- R3, R9: value 39k -> 47k

Commit message: Update board designs
Parts:
- removed the G*** at (52.9, 42.1)
- removed the G*** at (134.0, 51.4)
- added G***: LOGO, 4201_multiples:4201_V_0_2_0, F.Cu at (133.6, 51.4)
- added Ref**: Val**, 4201_multiples:4201_multiples_panel_silk, F.Cu at (50.7, 104.9)
- added Ref**: Val**, 4201_multiples:serial_no, B.Cu at (43.2, 104.8)
- C1, C2: value 47uF -> 22u
- R1, R7: value 220k -> 470k
- U1, U2: value TL074 -> LM324
Other:
- board text added: "4201 V0.2.0 INTERFACE"
- board text added: "4201 V0.2.0 MAIN BOARD"
- board text added: "4201 V0.2.0 PANEL"
