File: 4201_multiples_kicad/4201_multiples.kicad_sch (KiCad schematic)
At the start: 10 parts, among them J10 Conn_01x04_Female, J11 Conn_01x05_Female, J12 Conn_01x04_Female, J13 Conn_01x04_Female, J14 Conn_01x05_Male, J15 Conn_01x04_Male, J16 Conn_01x05_Male, J17 Conn_01x04_Male, J18 Conn_01x04_Male, J9 Conn_01x05_Female

Commit message: Small changes, cleanup
Connections:
- net interface/LED_1N_K renamed interface/LED_1P_K
- net interface/LED_1P_A renamed interface/LED_1N_A
- net interface/LED_1_PK_NA renamed interface/LED_1_PA_NK
- net interface/LED_2N_K renamed interface/LED_2P_K
- net interface/LED_2P_A renamed interface/LED_2N_A
- net interface/LED_2_PK_NA renamed interface/LED_2_PA_NK
- net main_board/LED_1N_K renamed main_board/LED_1P_K
- net main_board/LED_1P_A renamed main_board/LED_1N_A
- net main_board/LED_1_PK_NA renamed main_board/LED_1_PA_NK
- net main_board/LED_2N_K renamed main_board/LED_2P_K
- net main_board/LED_2P_A renamed main_board/LED_2N_A
- net main_board/LED_2_PK_NA renamed main_board/LED_2_PN_KA
Other:
- sheet interface ports: added LED_1N_A, LED_1P_K, LED_1_PA_NK, LED_2N_A, LED_2P_K, LED_2_PA_NK; removed LED_1N_K, LED_1P_A, LED_1_PK_NA, LED_2N_K, LED_2P_A, LED_2_PK_NA
- sheet main_board ports: added LED_1N_A, LED_1P_K, LED_1_PA_NK, LED_2N_A, LED_2P_K, LED_2_PN_KA; removed LED_1N_K, LED_1P_A, LED_1_PK_NA, LED_2N_K, LED_2P_A, LED_2_PK_NA
Changed lines of the file:
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@@
-      (effects (font (size 1.27 1.27)) (justify left))
-    )
-    (pin "LED_1_PK_NA" input (at 194.31 74.93 180)
-      (effects (font (size 1.27 1.27)) (justify left))
-    )
-    (pin "LED_1P_A" input (at 194.31 69.85 180)
-      (effects (font (size 1.27 1.27)) (justify left))
-    )
-    (pin "LED_1N_K" input (at 194.31 72.39 180)
-      (effects (font (size 1.27 1.27)) (justify left))
-    )
-    (pin "LED_2P_A" input (at 194.31 109.22 180)
-      (effects (font (size 1.27 1.27)) (justify left))
-    )
-    (pin "LED_2N_K" input (at 194.31 106.68 180)
-      (effects (font (size 1.27 1.27)) (justify left))
-    )
-    (pin "LED_2_PK_NA" input (at 194.31 104.14 180)
       (effects (font (size 1.27 1.27)) (justify left))
     )
     (pin "0V" input (at 194.31 49.53 180)
+      (effects (font (size 1.27 1.27)) (justify left))
+    )
+    (pin "LED_1P_K" input (at 194.31 72.39 180)
+      (effects (font (size 1.27 1.27)) (justify left))
+    )
+    (pin "LED_2_PN_KA" input (at 194.31 104.14 180)
+      (effects (font (size 1.27 1.27)) (justify left))
+    )
+    (pin "LED_2N_A" input (at 194.31 109.22 180)
+      (effects (font (size 1.27 1.27)) (justify left))
+    )
+    (pin "LED_2P_K" input (at 194.31 106.68 180)
+      (effects (font (size 1.27 1.27)) (justify left))
+    )
+    (pin "LED_1_PA_NK" input (at 194.31 74.93 180)
+      (effects (font (size 1.27 1.27)) (justify left))
+    )
+    (pin "LED_1N_A" input (at 194.31 69.85 180)
       (effects (font (size 1.27 1.27)) (justify left))
     )
@@
       (effects (font (size 1.27 1.27)) (justify right))
     )
-    (pin "LED_1P_A" input (at 87.63 69.85 0)
-      (effects (font (size 1.27 1.27)) (justify right))
-    )
-    (pin "LED_1N_K" input (at 87.63 72.39 0)
-      (effects (font (size 1.27 1.27)) (justify right))
-    )
-    (pin "LED_1_PK_NA" input (at 87.63 74.93 0)
-      (effects (font (size 1.27 1.27)) (justify right))
-    )
-    (pin "LED_2N_K" input (at 87.63 106.68 0)
-      (effects (font (size 1.27 1.27)) (justify right))
-    )
-    (pin "LED_2_PK_NA" input (at 87.63 104.14 0)
-      (effects (font (size 1.27 1.27)) (justify right))
-    )
-    (pin "LED_2P_A" input (at 87.63 109.22 0)
-      (effects (font (size 1.27 1.27)) (justify right))
-    )
     (pin "0V" input (at 87.63 49.53 0)
+      (effects (font (size 1.27 1.27)) (justify right))
+    )
+    (pin "LED_2_PA_NK" input (at 87.63 104.14 0)
+      (effects (font (size 1.27 1.27)) (justify right))
+    )
+    (pin "LED_2N_A" input (at 87.63 109.22 0)
+      (effects (font (size 1.27 1.27)) (justify right))
+    )
+    (pin "LED_1N_A" input (at 87.63 69.85 0)
+      (effects (font (size 1.27 1.27)) (justify right))
+    )
+    (pin "LED_1_PA_NK" input (at 87.63 74.93 0)
+      (effects (font (size 1.27 1.27)) (justify right))
+    )
+    (pin "LED_2P_K" input (at 87.63 106.68 0)
+      (effects (font (size 1.27 1.27)) (justify right))
+    )
+    (pin "LED_1P_K" input (at 87.63 72.39 0)
       (effects (font (size 1.27 1.27)) (justify right))
     )
@@
     )
     (path "/8b813b1d-c5b7-4977-8cc0-24b51b89bbdb/581392b2-5bd3-4fce-bbc9-6220495f2795"
-      (reference "D1") (unit 1) (value "1.8mm_green") (footprint "LED_THT:LED_D1.8mm_W3.3mm_H2.4mm")
+      (reference "D1") (unit 1) (value "1.8mm_red") (footprint "LED_THT:LED_D1.8mm_W3.3mm_H2.4mm")
     )
     (path "/8b813b1d-c5b7-4977-8cc0-24b51b89bbdb/158ad437-6a62-49f8-9c0c-193ea97af247"
-      (reference "D2") (unit 1) (value "1.8mm_red") (footprint "LED_THT:LED_D1.8mm_W3.3mm_H2.4mm")
+      (reference "D2") (unit 1) (value "1.8mm_green") (footprint "LED_THT:LED_D1.8mm_W3.3mm_H2.4mm")
     )
     (path "/8b813b1d-c5b7-4977-8cc0-24b51b89bbdb/bde82825-7270-4cab-a62e-613890f545c3"
-      (reference "D3") (unit 1) (value "1.8mm_green") (footprint "LED_THT:LED_D1.8mm_W3.3mm_H2.4mm")
+      (reference "D3") (unit 1) (value "1.8mm_red") (footprint "LED_THT:LED_D1.8mm_W3.3mm_H2.4mm")
     )
     (path "/8b813b1d-c5b7-4977-8cc0-24b51b89bbdb/6eda50de-002d-4e50-bdce-60c00143f3f0"
-      (reference "D4") (unit 1) (value "1.8mm_red") (footprint "LED_THT:LED_D1.8mm_W3.3mm_H2.4mm")
+      (reference "D4") (unit 1) (value "green") (footprint "LED_THT:LED_D1.8mm_W3.3mm_H2.4mm")
     )
     (path "/7cd117d0-9d7c-47f8-b2dc-5750ac60f5ae/295bc0c1-4fad-4cd1-abc2-3654cf56cfe4"
@@
     )
     (path "/8b813b1d-c5b7-4977-8cc0-24b51b89bbdb/a8cab53d-e2b5-4f13-a45d-cfd2eb662e0a"
-      (reference "J1") (unit 1) (value "AudioJack2") (footprint "OS_Connectors:Jack_3.5mm_PJ392_Vertical")
+      (reference "J1") (unit 1) (value "PJ392") (footprint "OS_Connectors:Jack_3.5mm_PJ392_Vertical")
     )
     (path "/8b813b1d-c5b7-4977-8cc0-24b51b89bbdb/fbf9af5e-6d0a-4bcd-94a8-7e4d105566b1"
-      (reference "J2") (unit 1) (value "AudioJack2") (footprint "OS_Connectors:Jack_3.5mm_PJ392_Vertical")
+      (reference "J2") (unit 1) (value "PJ392") (footprint "OS_Connectors:Jack_3.5mm_PJ392_Vertical")
     )
     (path "/8b813b1d-c5b7-4977-8cc0-24b51b89bbdb/b27e369e-6f41-474a-9a87-fe56295fd1f0"
-      (reference "J3") (unit 1) (value "AudioJack2") (footprint "OS_Connectors:Jack_3.5mm_PJ392_Vertical")
+      (reference "J3") (unit 1) (value "PJ392") (footprint "OS_Connectors:Jack_3.5mm_PJ392_Vertical")
     )
     (path "/8b813b1d-c5b7-4977-8cc0-24b51b89bbdb/b79720b9-7d33-4799-a13f-5c67646002e3"
-      (reference "J4") (unit 1) (value "AudioJack2") (footprint "OS_Connectors:Jack_3.5mm_PJ392_Vertical")
+      (reference "J4") (unit 1) (value "PJ392") (footprint "OS_Connectors:Jack_3.5mm_PJ392_Vertical")
     )
     (path "/8b813b1d-c5b7-4977-8cc0-24b51b89bbdb/d0a3249b-69ae-492c-b7ba-70d93167a06d"
-      (reference "J5") (unit 1) (value "AudioJack2") (footprint "OS_Connectors:Jack_3.5mm_PJ392_Vertical")
+      (reference "J5") (unit 1) (value "PJ392") (footprint "OS_Connectors:Jack_3.5mm_PJ392_Vertical")
     )
     (path "/8b813b1d-c5b7-4977-8cc0-24b51b89bbdb/08739723-018b-4ece-ae70-ea3c46ff72e3"
-      (reference "J6") (unit 1) (value "AudioJack2") (footprint "OS_Connectors:Jack_3.5mm_PJ392_Vertical")
+      (reference "J6") (unit 1) (value "PJ392") (footprint "OS_Connectors:Jack_3.5mm_PJ392_Vertical")
     )
     (path "/8b813b1d-c5b7-4977-8cc0-24b51b89bbdb/eb6fdb07-a946-482a-b267-ea225d0c19e8"
-      (reference "J7") (unit 1) (value "AudioJack2") (footprint "OS_Connectors:Jack_3.5mm_PJ392_Vertical")
+      (reference "J7") (unit 1) (value "PJ392") (footprint "OS_Connectors:Jack_3.5mm_PJ392_Vertical")
     )
     (path "/8b813b1d-c5b7-4977-8cc0-24b51b89bbdb/4afd2d19-3ce6-44d7-9813-913e5ac19fd0"
-      (reference "J8") (unit 1) (value "AudioJack2") (footprint "OS_Connectors:Jack_3.5mm_PJ392_Vertical")
+      (reference "J8") (unit 1) (value "PJ392") (footprint "OS_Connectors:Jack_3.5mm_PJ392_Vertical")
     )
     (path "/d75952f5-86ee-4cc5-8635-c8cf434a5fd0"
