File: 4201_multiples_kicad/main_board.kicad_sch (KiCad schematic)
At the start: 31 parts, among them J19 Conn_02x05_Odd_Even, U1 LM324, U2 LM324

Commit message: Update some smybols and run all checks
Parts:
- D10, D11, D12, D13, D14, D5, D6, D7, D8, D9: footprint Diode_SMD:D_1206_3216Metric_Pad1.42x1.75mm_HandSolder -> Diode_THT:D_DO-41_SOD81_P10.16mm_Horizontal
Changed lines of the file:
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@@
     (pin "1")
   )
-  (symbol (lib_id "Diode:1N4007") (at 195.58 76.2 180) (unit 1)
+  (symbol (lib_name "1N4007_2") (lib_id "Diode:1N4007") (at 195.58 76.2 180) (unit 1)
     (in_bom yes) (on_board yes)
     (property "Reference" "D5" (id 0) (at 194.31 80.01 0)
@@
       (effects (font (size 1.27 1.27)) (justify right))
     )
-    (property "Footprint" "Diode_SMD:D_1206_3216Metric_Pad1.42x1.75mm_HandSolder" (id 2) (at 195.58 71.755 0)
+    (property "Footprint" "Diode_THT:D_DO-41_SOD81_P10.16mm_Horizontal" (id 2) (at 195.58 71.755 0)
       (effects (font (size 1.27 1.27)) hide)
     )
@@
     (property "Reference" "D13" (id 0) (at 56.1975 139.7 0))
     (property "Value" "LL103A" (id 1) (at 56.1975 142.24 0))
-    (property "Footprint" "Diode_SMD:D_1206_3216Metric_Pad1.42x1.75mm_HandSolder" (id 2) (at 55.88 141.605 0)
+    (property "Footprint" "Diode_THT:D_DO-41_SOD81_P10.16mm_Horizontal" (id 2) (at 55.88 141.605 0)
       (effects (font (size 1.27 1.27)) hide)
     )
@@
     (pin "1")
   )
-  (symbol (lib_id "Diode:1N4007") (at 187.96 106.68 270) (unit 1)
+  (symbol (lib_name "1N4007_4") (lib_id "Diode:1N4007") (at 187.96 106.68 270) (unit 1)
     (in_bom yes) (on_board yes)
     (property "Reference" "D8" (id 0) (at 193.04 106.68 90)
@@
       (effects (font (size 1.27 1.27)) (justify right))
     )
-    (property "Footprint" "Diode_SMD:D_1206_3216Metric_Pad1.42x1.75mm_HandSolder" (id 2) (at 183.515 106.68 0)
+    (property "Footprint" "Diode_THT:D_DO-41_SOD81_P10.16mm_Horizontal" (id 2) (at 183.515 106.68 0)
       (effects (font (size 1.27 1.27)) hide)
     )
@@
     (pin "2")
   )
-  (symbol (lib_id "Diode:1N4007") (at 232.41 106.68 90) (unit 1)
+  (symbol (lib_name "1N4007_1") (lib_id "Diode:1N4007") (at 232.41 106.68 90) (unit 1)
     (in_bom yes) (on_board yes)
     (property "Reference" "D11" (id 0) (at 234.95 106.68 90)
@@
       (effects (font (size 1.27 1.27)) (justify right))
     )
-    (property "Footprint" "Diode_SMD:D_1206_3216Metric_Pad1.42x1.75mm_HandSolder" (id 2) (at 236.855 106.68 0)
+    (property "Footprint" "Diode_THT:D_DO-41_SOD81_P10.16mm_Horizontal" (id 2) (at 236.855 106.68 0)
       (effects (font (size 1.27 1.27)) hide)
     )
@@
     (pin "2")
   )
-  (symbol (lib_id "Diode:1N4007") (at 195.58 62.23 0) (unit 1)
+  (symbol (lib_name "1N4007_3") (lib_id "Diode:1N4007") (at 195.58 62.23 0) (unit 1)
     (in_bom yes) (on_board yes)
     (property "Reference" "D6" (id 0) (at 196.85 67.31 0)
@@
       (effects (font (size 1.27 1.27)) (justify right))
     )
-    (property "Footprint" "Diode_SMD:D_1206_3216Metric_Pad1.42x1.75mm_HandSolder" (id 2) (at 195.58 66.675 0)
+    (property "Footprint" "Diode_THT:D_DO-41_SOD81_P10.16mm_Horizontal" (id 2) (at 195.58 66.675 0)
       (effects (font (size 1.27 1.27)) hide)
     )
@@
       (effects (font (size 1.27 1.27)) (justify right))
     )
-    (property "Footprint" "Diode_SMD:D_1206_3216Metric_Pad1.42x1.75mm_HandSolder" (id 2) (at 240.665 106.68 0)
+    (property "Footprint" "Diode_THT:D_DO-41_SOD81_P10.16mm_Horizontal" (id 2) (at 240.665 106.68 0)
       (effects (font (size 1.27 1.27)) hide)
     )
@@
     (property "Reference" "D14" (id 0) (at 55.5625 149.86 0))
     (property "Value" "LL103A" (id 1) (at 55.5625 152.4 0))
-    (property "Footprint" "Diode_SMD:D_1206_3216Metric_Pad1.42x1.75mm_HandSolder" (id 2) (at 55.88 160.655 0)
+    (property "Footprint" "Diode_THT:D_DO-41_SOD81_P10.16mm_Horizontal" (id 2) (at 55.88 160.655 0)
       (effects (font (size 1.27 1.27)) hide)
     )
@@
     (pin "4")
   )
-  (symbol (lib_id "Diode:1N4007") (at 252.73 76.2 180) (unit 1)
+  (symbol (lib_name "1N4007_6") (lib_id "Diode:1N4007") (at 252.73 76.2 180) (unit 1)
     (in_bom yes) (on_board yes)
     (property "Reference" "D9" (id 0) (at 251.46 80.01 0)
@@
       (effects (font (size 1.27 1.27)) (justify right))
     )
-    (property "Footprint" "Diode_SMD:D_1206_3216Metric_Pad1.42x1.75mm_HandSolder" (id 2) (at 252.73 71.755 0)
+    (property "Footprint" "Diode_THT:D_DO-41_SOD81_P10.16mm_Horizontal" (id 2) (at 252.73 71.755 0)
       (effects (font (size 1.27 1.27)) hide)
     )
@@
     (pin "1")
   )
-  (symbol (lib_id "Diode:1N4007") (at 175.26 106.68 90) (unit 1)
+  (symbol (lib_name "1N4007_5") (lib_id "Diode:1N4007") (at 175.26 106.68 90) (unit 1)
     (in_bom yes) (on_board yes)
     (property "Reference" "D7" (id 0) (at 177.8 106.68 90)
@@
       (effects (font (size 1.27 1.27)) (justify right))
     )
-    (property "Footprint" "Diode_SMD:D_1206_3216Metric_Pad1.42x1.75mm_HandSolder" (id 2) (at 179.705 106.68 0)
+    (property "Footprint" "Diode_THT:D_DO-41_SOD81_P10.16mm_Horizontal" (id 2) (at 179.705 106.68 0)
       (effects (font (size 1.27 1.27)) hide)
     )
@@
     (pin "1")
   )
-  (symbol (lib_id "Diode:1N4007") (at 252.73 62.23 0) (unit 1)
+  (symbol (lib_name "1N4007_7") (lib_id "Diode:1N4007") (at 252.73 62.23 0) (unit 1)
     (in_bom yes) (on_board yes)
     (property "Reference" "D10" (id 0) (at 254 67.31 0)
@@
       (effects (font (size 1.27 1.27)) (justify right))
     )
-    (property "Footprint" "Diode_SMD:D_1206_3216Metric_Pad1.42x1.75mm_HandSolder" (id 2) (at 252.73 66.675 0)
-      (effects (font (size 1.27 1.27)) hide)
-    )
+    (property "Footprint" "Diode_THT:D_DO-41_SOD81_P10.16mm_Horizontal" (id 2) (at 252.73 66.675 0)
+      (effects (font (size 1.27 1.27)) hide)
+    )
